File: RTx_Controller_Board/RTxController.brd (EAGLE design)
At the start: 161.3 x 55.9 mm, 214 parts, among them IC1 LTC4263, IC2 TLK110", J22 Debug Header, SW1 COM08720, U1 STM32F407ZXT, U2 TPD4S012, X4 MINI-USB-32005-301, X8 0826-1X1T-GJ-F

Commit message: updated layout of Rtx Controller Board.
Parts:
- removed C100, C105, C106, C107, C108, C113, C114, C115, C116, C121, C122, C123, C124, C97, C98, C99: NU, motorFeedback:C0603
- moved R53 839.0 mm to (65.3, 44.7)
- moved R52 837.1 mm to (65.3, 47.5)
- moved R51 815.5 mm to (81.5, 24.1), turned to 90 degrees
- moved R48 812.6 mm to (91.2, 27.2), turned to 90 degrees
- moved R49 810.3 mm to (79.5, 24.1), turned to 90 degrees
- moved R44 807.7 mm to (71.4, 48.3), turned to 180 degrees
- moved R47 806.8 mm to (88.9, 26.7), turned to 90 degrees
- moved R46 801.0 mm to (86.6, 26.2), turned to 90 degrees
- moved R43 800.9 mm to (71.4, 46.0), turned to 180 degrees
- moved R45 795.2 mm to (84.3, 25.7), turned to 90 degrees
- moved R42 794.4 mm to (71.9, 43.7), turned to 180 degrees
- moved R41 787.9 mm to (72.6, 41.4), turned to 180 degrees
- moved R40 779.2 mm to (84.1, 32.8), turned to 270 degrees
- moved R39 774.8 mm to (86.6, 32.0), turned to 270 degrees
- moved R54 771.2 mm to (124.0, 46.2), turned to 180 degrees
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Connections:
- net +5.000VREF: now also X1.10, X1.13, X1.9; no longer X1.12, X1.2, X1.3
- net ENABLE_AXIS3_OUT: no longer C116.1
- net ENABLE_AXIS4_OUT: no longer C114.1
- net ENABLE_LAT_OUT: no longer C107.1
- net ENABLE_VERT_OUT: no longer C105.1
- net GND: no longer C100.2, C105.2, C106.2, C107.2, C108.2, C113.2, C114.2, C115.2, C116.2, C121.2, C122.2, C123.2, C124.2, C97.2, C98.2, C99.2
- net N$14: now also X1.2; no longer X1.4
- net N$6: now also X1.4; no longer X1.15
- net N$9: now also X1.3; no longer X1.11
- net PWM_AXIS3_U_OUT: no longer C123.1
- net PWM_AXIS3_V_OUT: no longer C124.1
- net PWM_AXIS4_U_OUT: no longer C121.1
- net PWM_AXIS4_V_OUT: no longer C122.1
- net PWM_LAT_U_OUT: no longer C97.1
- net PWM_LAT_V_OUT: no longer C98.1
- net PWM_VERT_U_OUT: no longer C99.1
- net PWM_VERT_V_OUT: no longer C100.1
- net WATCHDOG_AXIS3_OUT: no longer C115.1
- net WATCHDOG_AXIS4_OUT: no longer C113.1
- net WATCHDOG_LAT_OUT: no longer C108.1
- net WATCHDOG_VERT_OUT: no longer C106.1
Routing:
- net +5.000VREF: track 0.00 -> 56.0 mm
- net +3.3V: track 7.19 -> 49.5 mm
- net PWM_AXIS3_V_OUT: track 0.00 -> 17.3 mm
- net PWM_LAT_U_OUT: track 0.00 -> 17.1 mm
- net NRST: track 0.00 -> 15.2 mm
- net PWM_AXIS3_U_OUT: track 0.00 -> 15.0 mm
- net PWM_LAT_V_OUT: track 0.00 -> 14.8 mm
- net N$6: track 0.00 -> 13.7 mm
- net PWM_VERT_U_OUT: track 0.00 -> 12.9 mm
- net PWM_AXIS4_V_OUT: track 0.00 -> 12.8 mm
- net ADC2_IN+: track 0.00 -> 12.8 mm
- net ADC4_IN: track 0.00 -> 12.7 mm
- net WATCHDOG_AXIS4_OUT: track 0.00 -> 12.4 mm
- net WATCHDOG_VERT_OUT: track 0.00 -> 11.4 mm
- net ADC3_IN+: track 0.00 -> 10.5 mm
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- added copper zone on layer 1, net GND
Other:
- board size 161.3 x 55.9 mm -> 161.3 x 90.2 mm

Commit message: Ethernet and PoE controllers completely redone.
Parts:
- removed C43, C47: 0.1u 100v, motorFeedback:C0805K
- removed C49: 0.1uf, motorFeedback:C0805K
- removed C52, C53: 1u, motorFeedback:C0805K
- removed C56, C57, C58, C59, C60, C61, C62, C63, C64, C65, C66, C67, C68, C69, C70, C71: (no value), motorFeedback:C0805K
- removed D1: SMAJ58A, diode:SMBJ
- removed D2: MMBD6050LT1SOT23, motorFeedback:SOT23-TO-236
- removed F1: 1A, special:FUSE
- removed IC1: LTC4263, motorFeedback:S14-NARROW
- removed JP1: NU, motorFeedback:1X06
- removed L1: 10m, 21mA, motorFeedback:0204V
- removed LED1: (no value), motorFeedback:LED5MM
- removed R25, R28: 470, motorFeedback:R0603
- removed R26: 4.87k, motorFeedback:R0603
- removed R27, R29, R32: 2.2k, motorFeedback:R0603
- removed R30: 49.9, motorFeedback:R0603
- removed R31, R33, R34, R35, R_LED1: 1k, motorFeedback:R0603
- added C54, C75, C76, C98, C99: 100n, rcl_custom:0402-C-NOSILK
- added C73, C97: 22u, rcl_custom:1206-C
- added C77: 2.2u, rcl_custom:0402-C-NOSILK
- added D3, D5: 1N4448, temp_library:SOD-123
- added D4: SMAJ58A, diode:SMBJ
- added L2: 10m, 21mA, motorFeedback:0204V
- added L3: FB0805/600R/200mA(201209-601), rcl_custom:0805-C-NOSILK
- added R55, R56, R59: 1k, rcl_custom:0402-C-NOSILK
- added R60: 6.49k, rcl_custom:0402-C-NOSILK
- added R99: 2.2M, motorFeedback:R0603
- added U3: KSZ8081, ksz8081:QFN-24
- C44: value 1u -> 100nF
- C48, C51: value 0.1u -> 0.1uf 100V
- C50: value 1u -> 47uf 100V
- IC2: value TLK110" -> MAX5984C; device motorFeedback:LQFP48 -> temp_library:TQFN-28
- R24: value 49.9 -> 1k
- R54: device rcl:RTRIM4G/J -> pot:3223W
- moved R24 1089.5 mm to (-216.9, -967.5)
- moved R23 1087.3 mm to (-216.9, -962.7)
- moved C51 1067.9 mm to (-210.3, -953.0), turned to 0 degrees
- moved C50 1059.9 mm to (-195.3, -948.2)
- moved C48 1057.2 mm to (-195.3, -943.4), turned to 0 degrees
- moved C44 1041.3 mm to (-195.3, -927.9), turned to 0 degrees
- moved IC2 1037.6 mm to (-194.1, -922.5), turned to 0 degrees
- moved R_LED 713.0 mm to (-195.6, -932.7)
Connections:
- removed net N$23: L1.2, LED1.K
- removed net N$24: D2.1, L1.1, R_LED.2, R_LED1.2
- removed net N$25: IC1.1, R_LED.1, R_LED1.1
- removed net N$31: IC2.21, R33.1
- removed net N$32: R28.2, X8.19
- removed net N$33: IC2.28, R25.1, R29.1
- removed net N$37: IC2.29, R34.1
- removed net N$38: IC2.7, R35.1
- removed net N$40: IC2.24, R26.2
- removed net N$41: C68.2, C69.2, C70.2, C71.2, IC2.18, IC2.23, IC2.37
- removed net N$56: IC2.8, JP1.1
- removed net N$57: IC2.12, JP1.2
- removed net N$58: IC2.9, JP1.3
- removed net N$59: IC2.10, JP1.4
- removed net N$60: IC2.11, JP1.5
- removed net PORT_MAGNETICS+: C47.1, F1.2, X8.15
- removed net PORT_MAGNETICS-: C47.2, D1.A, IC1.10, IC1.9, X8.16
- new net ACTIVITY_LED: R59.1, U3.23
- new net EPHY_NRST: U3.24
- new net ETH_CRS_DV: U3.15
- new net ETH_MDINT: R56.2, U3.18
- new net ETH_RMII_REF_CLK: U3.16
- new net ETH_RXD0: U3.13
- new net ETH_RXD1: U3.12
- new net ETH_TXD0: U3.20
- new net ETH_TXD1: U3.21
- new net ETH_TX_EN: U3.19
- new net MCO1-ETH-CLK: U3.8
- new net N$21: U3.6, X8.11
- new net N$30: C44.1, IC2.14
- new net N$79: R60.2, U3.9
- new net N$80: C76.1, C77.1, U3.1
- new net N$82: C99.2, X8.12
- new net POE_LED+: L2.1, X8.17
- new net POE_LED-: D3.P$1, R_LED.2, X8.18
- new net PSE_OUTPUT: C51.2, D4.A, D5.P$1, IC2.25, IC2.26, IC2.27, R99.2, X8.14
- new net VDDA: C54.2, X8.6
- new net VDDA_3.3: C97.2, C98.2, L3.1, U3.2
- net +3.3V: now also C73.2, C75.2, L3.2, R55.1, R56.1, U3.14, X8.19; no longer C44.1, C48.1, C50.1, C51.1, C52.1, C53.1, C56.2, C57.2, C58.2, C59.2, C60.2, C61.2, C62.2, C63.2, C64.2, C65.2, C66.2, C67.2, IC2.22, IC2.32, IC2.48, R23.1, R24.2, R27.1, R30.2, R31.1, R33.2, R34.2, R35.2, X8.12, X8.6
- net ETH_MCO1: no longer IC2.34
- net ETH_MDC: now also U3.11; no longer IC2.31
- net ETH_MDIO: now also R55.2, U3.10; no longer IC2.30
- net ETH_MII_COL: no longer IC2.42
- net ETH_MII_CRS: no longer IC2.40
- net ETH_MII_RXD0: no longer IC2.43
- net ETH_MII_RXD1: no longer IC2.44
- net ETH_MII_RXD2: no longer IC2.45
- net ETH_MII_RXD3: no longer IC2.46
- net ETH_MII_RX_CLK: no longer IC2.38
- net ETH_MII_RX_DV: no longer IC2.39
- net ETH_MII_RX_ER: no longer IC2.41
- net ETH_MII_TXD0: no longer IC2.3
- net ETH_MII_TXD1: no longer IC2.4
- net ETH_MII_TXD2: no longer IC2.5
- net ETH_MII_TXD3: no longer IC2.6
- net ETH_MII_TX_CLK: no longer IC2.1
- net ETH_MII_TX_EN: no longer IC2.2
- net GND: now also C54.1, C73.1, C75.1, C76.2, C77.2, C97.1, C98.1, C99.1, R60.1, U3.22, U3.PAD; no longer C44.2, C48.2, C50.2, C51.2, C52.2, C53.2, C56.1, C57.1, C58.1, C59.1, C60.1, C61.1, C62.1, C63.1, C64.1, C65.1, C66.1, C67.1, C68.1, C69.1, C70.1, C71.1, IC2.15, IC2.19, IC2.35, IC2.36, IC2.47, JP1.6, R26.1, R29.2, R32.2, X8.18, X8.20
- net N$15: now also R59.2, X8.20; no longer C49.1, IC1.12, IC1.13, IC1.14
- net N$26: now also U3.5, X8.10; no longer IC2.17, R23.2, X8.11
- net N$27: now also U3.4, X8.4; no longer IC2.16, R24.1, X8.10
- net N$28: now also U3.3, X8.5; no longer IC2.14, R31.2, X8.4
- net N$29: now also IC2.17, R_LED.1; no longer IC2.13, R30.1, X8.5
- net N$34: now also D5.P$2, IC2.23; no longer IC2.20, R27.2
- net N$35: now also IC2.4, R23.1; no longer R25.2, X8.17
- net N$36: now also IC2.5, R24.1; no longer IC2.27, R28.1, R32.1
- net POE+: now also C48.1, C50.1, C51.1, D3.P$2, D4.C, IC2.21, L2.2, R99.1, X8.13; no longer C43.1, D1.C, D2.3, F1.1, IC1.11, LED1.A
- net POE-: now also C44.2, C48.2, C50.2, IC2.1, IC2.10, IC2.11, IC2.12, IC2.13, IC2.15, IC2.19, IC2.2, IC2.3, IC2.7, IC2.8, IC2.9, IC2.PAD, R23.2, R24.2; no longer C43.2, C49.2, IC1.2, IC1.3, IC1.4, IC1.5, IC1.6, IC1.7

Commit message: Ethernet pinout.
Connections:
- removed net ETH_MCO1: U1.67
- removed net ETH_MII_COL: U1.26
- removed net ETH_MII_CRS: U1.23
- removed net ETH_MII_RXD0: U1.33
- removed net ETH_MII_RXD1: U1.34
- removed net ETH_MII_RXD2: U1.35
- removed net ETH_MII_RXD3: U1.36
- removed net ETH_MII_RX_CLK: U1.24
- removed net ETH_MII_RX_DV: U1.32
- removed net ETH_MII_RX_ER: U1.47
- removed net ETH_MII_TXD0: U1.51
- removed net ETH_MII_TXD1: U1.52
- removed net ETH_MII_TXD2: U1.17
- removed net ETH_MII_TXD3: U1.95
- removed net ETH_MII_TX_CLK: U1.18
- removed net ETH_MII_TX_EN: U1.48
- net EPHY_NRST: now also U1.97
- net ETH_CRS_DV: now also U1.32
- net ETH_MDINT: now also U1.26
- net ETH_RMII_REF_CLK: now also U1.24
- net ETH_RXD0: now also U1.33
- net ETH_RXD1: now also U1.34
- net ETH_TXD0: now also U1.51
- net ETH_TXD1: now also U1.52
- net ETH_TX_EN: now also U1.48
- net MCO1-ETH-CLK: now also U1.67
Changed lines of the file:
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@@
 <wire x1="106.172" y1="52.07" x2="141.986" y2="76.454" width="0" layer="19" extent="1-1"/>
-</signal>
-<signal name="ETH_MII_RX_CLK">
-<contactref element="U1" pad="24"/>
-</signal>
-<signal name="ETH_MII_RX_DV">
-<contactref element="U1" pad="32"/>
-</signal>
-<signal name="ETH_MII_RX_ER">
-<contactref element="U1" pad="47"/>
-</signal>
-<signal name="ETH_MII_RXD0">
-<contactref element="U1" pad="33"/>
-</signal>
-<signal name="ETH_MII_RXD1">
-<contactref element="U1" pad="34"/>
-</signal>
-<signal name="ETH_MII_RXD2">
-<contactref element="U1" pad="35"/>
-</signal>
-<signal name="ETH_MII_RXD3">
-<contactref element="U1" pad="36"/>
-</signal>
-<signal name="ETH_MII_TX_CLK">
-<contactref element="U1" pad="18"/>
-</signal>
-<signal name="ETH_MII_TX_EN">
-<contactref element="U1" pad="48"/>
-</signal>
-<signal name="ETH_MII_TXD0">
-<contactref element="U1" pad="51"/>
-</signal>
-<signal name="ETH_MII_TXD1">
-<contactref element="U1" pad="52"/>
-</signal>
-<signal name="ETH_MII_TXD2">
-<contactref element="U1" pad="17"/>
-</signal>
-<signal name="ETH_MII_TXD3">
-<contactref element="U1" pad="95"/>
-</signal>
-<signal name="ETH_MII_CRS">
-<contactref element="U1" pad="23"/>
-</signal>
-<signal name="ETH_MII_COL">
-<contactref element="U1" pad="26"/>
 </signal>
 <signal name="ETH_MDC">
@@
 <wire x1="39.766" y1="18.288" x2="63.048" y2="21.236" width="0" layer="19" extent="1-1"/>
 </signal>
-<signal name="ETH_MCO1">
-<contactref element="U1" pad="67"/>
-</signal>
 <signal name="N$43">
 <contactref element="R36" pad="2"/>
@@
 <signal name="ETH_CRS_DV">
 <contactref element="U3" pad="15"/>
+<contactref element="U1" pad="32"/>
+<wire x1="-170.692" y1="-893.998" x2="63.548" y2="21.236" width="0" layer="19" extent="1-1"/>
 </signal>
 <signal name="ETH_RXD0">
 <contactref element="U3" pad="13"/>
+<contactref element="U1" pad="33"/>
+<wire x1="-169.692" y1="-893.998" x2="64.048" y2="21.236" width="0" layer="19" extent="1-1"/>
 </signal>
 <signal name="ETH_RXD1">
 <contactref element="U3" pad="12"/>
+<contactref element="U1" pad="34"/>
+<wire x1="-169.082" y1="-894.608" x2="64.548" y2="21.236" width="0" layer="19" extent="1-1"/>
 </signal>
 <signal name="EPHY_NRST">
 <contactref element="U3" pad="24"/>
+<contactref element="U1" pad="97"/>
+<wire x1="-172.802" y1="-897.108" x2="62.048" y2="36.676" width="0" layer="19" extent="1-1"/>
 </signal>
 <signal name="ETH_TX_EN">
 <contactref element="U3" pad="19"/>
+<contactref element="U1" pad="48"/>
+<wire x1="-172.802" y1="-894.608" x2="71.548" y2="21.236" width="0" layer="19" extent="1-1"/>
 </signal>
 <signal name="ETH_TXD0">
 <contactref element="U3" pad="20"/>
+<contactref element="U1" pad="51"/>
+<wire x1="-172.802" y1="-895.108" x2="74.268" y2="22.956" width="0" layer="19" extent="1-1"/>
 </signal>
 <signal name="ETH_TXD1">
 <contactref element="U3" pad="21"/>
+<contactref element="U1" pad="52"/>
+<wire x1="-172.802" y1="-895.608" x2="74.268" y2="23.456" width="0" layer="19" extent="1-1"/>
 </signal>
 <signal name="ETH_MDINT">
 <contactref element="R56" pad="2"/>
 <contactref element="U3" pad="18"/>
+<contactref element="U1" pad="26"/>
+<wire x1="-183.72" y1="-905.002" x2="60.548" y2="21.236" width="0" layer="19" extent="1-1"/>
 <wire x1="-172.192" y1="-893.998" x2="-183.72" y2="-905.002" width="0" layer="19" extent="1-1"/>
 </signal>
@@
 <signal name="ETH_RMII_REF_CLK">
 <contactref element="U3" pad="16"/>
+<contactref element="U1" pad="24"/>
+<wire x1="-171.192" y1="-893.998" x2="58.828" y2="23.456" width="0" layer="19" extent="1-1"/>
 </signal>
 <signal name="MCO1-ETH-CLK">
 <contactref element="U3" pad="8"/>
+<contactref element="U1" pad="67"/>
+<wire x1="-169.082" y1="-896.608" x2="74.268" y2="30.956" width="0" layer="19" extent="1-1"/>
 </signal>
 <signal name="N$79">

Commit message: Added LEDs and testpoints to processor for debugging. Fixed JTAG connector.
Parts:
- removed R168: 100, rcl_custom:0402-B-NOSILK
- removed TP38: TPTP06R, testpad:TP06R
- added LED1: (no value), LED_RGB_PLCC6:PLCC-6
- added LED2, LED3, LED4, LED5: (no value), led:CHIP-LED0603
- added R25, R26, R27, R28, R29, R30, R31: 750, rcl:R0402
- added TP1, TP2, TP3, TP4, TP5, TP6, TP7: TPTP06R, testpad:TP06R
Connections:
- removed net N$206: J22.VTREF, R168.1
- removed net N$210: J22.GNDDET, TP38.TP
- new net N$23: LED2.A, R28.2
- new net N$24: LED3.A, R29.2
- new net N$25: LED1.3, R26.2
- new net N$31: LED1.4, R25.2
- new net N$32: LED1.1, R27.2
- new net N$33: TP6.TP, U1.53
- new net N$37: TP3.TP, U1.80
- new net N$38: TP4.TP, U1.8
- new net N$39: TP5.TP, U1.41
- new net N$40: TP2.TP, U1.3
- new net N$41: TP1.TP, U1.1
- new net N$44: TP7.TP, U1.23
- new net N$56: LED4.A, R30.2
- new net N$57: LED5.A, R31.2
- new net N$58: LED1.5, U1.40
- new net N$59: LED1.2, U1.42
- new net N$60: LED1.6, U1.44
- new net N$68: LED5.C, U1.5
- new net N$69: LED4.C, U1.4
- new net N$70: LED3.C, U1.2
- new net N$71: LED2.C, U1.98
- net +3.3V: now also J22.VTREF, R25.1, R26.1, R27.1, R28.1, R29.1, R30.1, R31.1; no longer R168.2
- net GND: now also J22.GNDDET
Routing:
- net N$206: track 3.37 -> 0.00 mm
- net +3.3V: track 49.5 -> 46.9 mm

Commit message: Updated USB portion of schematic to include crystal and fixed capacitance. Initial check in of crystal datasheet.
Parts:
- added C43: 16p, rcl:C0402
- added XTAL1: ABM8G, motorFeedback:ABM8G
- C45: value 10u -> 16p
- moved C45 1153.4 mm to (-246.9, -1033.0)
Connections:
- new net OSC_IN: C43.1, U1.12, XTAL1.1
- new net OSC_OUT: C45.1, U1.13, XTAL1.3
- net GND: now also C43.2
- net USB_VBUS: no longer C45.1
Changed lines of the file:
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@@
 <attribute name="OC_FARNELL" value="unknown" x="58.42" y="85.598" size="1.778" layer="27" rot="R270" display="off"/>
 </element>
-<element name="C45" library="rcl" package="C0402" value="10u" x="61.214" y="78.486"/>
 <element name="R21" library="rcl" package="R0402" value="22" x="51.816" y="75.184" rot="R180"/>
 <element name="R22" library="rcl" package="R0402" value="22" x="51.816" y="76.454" rot="R180"/>
@@
 <element name="R30" library="rcl" package="R0402" value="750" x="-242.57" y="-1019.81"/>
 <element name="R31" library="rcl" package="R0402" value="750" x="-242.57" y="-1024.636"/>
+<element name="XTAL1" library="motorFeedback" package="ABM8G" value="ABM8G" x="-246.126" y="-1023.874"/>
+<element name="C43" library="rcl" package="C0402" value="16p" x="-246.888" y="-1029.462"/>
+<element name="C45" library="rcl" package="C0402" value="16p" x="-246.888" y="-1033.018"/>
 </elements>
 <signals>
@@
 <contactref element="ADC4" pad="5"/>
 <contactref element="REF1" pad="4"/>
-<contactref element="C45" pad="2"/>
 <contactref element="X4" pad="5"/>
 <contactref element="U2" pad="4"/>
@@
 <contactref element="C98" pad="1"/>
 <contactref element="J22" pad="GNDDET"/>
+<contactref element="C43" pad="2"/>
+<contactref element="C45" pad="2"/>
 <wire x1="-188.326" y1="-810.26" x2="-188.326" y2="-814.832" width="0" layer="19" extent="1-1"/>
 <wire x1="-195.91" y1="-824.992" x2="-188.326" y2="-814.832" width="0" layer="19" extent="1-1"/>
@@
 <wire x1="-172.802" y1="-896.108" x2="-173.912" y2="-900.43" width="0" layer="19" extent="1-1"/>
 <wire x1="-170.942" y1="-895.858" x2="-172.802" y2="-896.108" width="0" layer="19" extent="1-1"/>
+<wire x1="-246.238" y1="-1029.462" x2="-196.01" y2="-905.002" width="0" layer="19" extent="1-1"/>
+<wire x1="-246.238" y1="-1033.018" x2="-246.238" y2="-1029.462" width="0" layer="19" extent="1-1"/>
 <wire x1="-119.038" y1="-612.14" x2="-188.326" y2="-810.26" width="0" layer="19" extent="1-1"/>
 <wire x1="37.454" y1="7.62" x2="-119.038" y2="-612.14" width="0" layer="19" extent="1-1"/>
@@
 <wire x1="154.0764" y1="37.338" x2="146.7612" y2="37.338" width="0" layer="19" extent="1-1"/>
 <wire x1="146.228" y1="46.482" x2="146.7612" y2="37.338" width="0" layer="19" extent="1-1"/>
-<wire x1="61.864" y1="78.486" x2="59.094" y2="47.498" width="0" layer="19" extent="1-1"/>
-<wire x1="61.864" y1="79.502" x2="61.864" y2="78.486" width="0" layer="19" extent="1-1"/>
-<wire x1="57.666" y1="79.394" x2="61.864" y2="79.502" width="0" layer="19" extent="1-1"/>
+<wire x1="57.666" y1="79.394" x2="59.094" y2="47.498" width="0" layer="19" extent="1-1"/>
 <wire x1="56.82" y1="82.598" x2="57.666" y2="79.394" width="0" layer="19" extent="1-1"/>
+<wire x1="61.864" y1="79.502" x2="57.666" y2="79.394" width="0" layer="19" extent="1-1"/>
 </signal>
 <signal name="+5V" airwireshidden="yes">
@@
 <contactref element="X4" pad="1"/>
 <contactref element="U2" pad="6"/>
-<contactref element="C45" pad="1"/>
 <contactref element="C46" pad="1"/>
 <contactref element="U1" pad="68"/>
-<wire x1="58.666" y1="79.394" x2="60.02" y2="82.598" width="0" layer="19" extent="1-1"/>
-<wire x1="60.564" y1="79.502" x2="58.666" y2="79.394" width="0" layer="19" extent="1-1"/>
-<wire x1="60.564" y1="78.486" x2="60.564" y2="79.502" width="0" layer="19" extent="1-1"/>
-<wire x1="74.268" y1="31.456" x2="58.666" y2="79.394" width="0" layer="19" extent="1-1"/>
+<wire x1="60.564" y1="79.502" x2="60.02" y2="82.598" width="0" layer="19" extent="1-1"/>
+<wire x1="58.666" y1="79.394" x2="60.564" y2="79.502" width="0" layer="19" extent="1-1"/>
+<wire x1="74.268" y1="31.456" x2="60.564" y2="79.502" width="0" layer="19" extent="1-1"/>
 </signal>
 <signal name="USB_D-">
@@
 <wire x1="61.548" y1="36.676" x2="-227.33" y2="-1005.598" width="0" layer="19" extent="1-1"/>
 </signal>
+<signal name="OSC_IN">
+<contactref element="U1" pad="12"/>
+<contactref element="C43" pad="1"/>
+<contactref element="XTAL1" pad="1"/>
+<wire x1="-247.538" y1="-1029.462" x2="58.828" y2="29.456" width="0" layer="19" extent="1-1"/>
+<wire x1="-247.226" y1="-1024.724" x2="-247.538" y2="-1029.462" width="0" layer="19" extent="1-1"/>
+</signal>
+<signal name="OSC_OUT">
+<contactref element="U1" pad="13"/>
+<contactref element="XTAL1" pad="3"/>
+<contactref element="C45" pad="1"/>
+<wire x1="-247.538" y1="-1033.018" x2="-245.026" y2="-1023.024" width="0" layer="19" extent="1-1"/>
+<wire x1="58.828" y1="28.956" x2="-245.026" y2="-1023.024" width="0" layer="19" extent="1-1"/>
+</signal>
 </signals>

Commit message: small changes made to layout.
Routing:
- net +5.000VREF: track 56.0 -> 84.9 mm, vias 0 -> 4
- net SPI_SCK: track 4.36 -> 26.6 mm, vias 0 -> 2
- net SDO3: track 0.00 -> 11.8 mm
- net VIO: track 3.87 -> 13.4 mm
- net SPI_NSS: track 0.00 -> 9.49 mm, vias 0 -> 2
- net N$67: track 7.86 -> 0.00 mm
- net N$66: track 7.86 -> 0.00 mm

Commit message: updates made to PCB layout
Parts:
- moved C45 1142.9 mm to (12.7, 80.0), turned to 270 degrees
- moved C43 1137.4 mm to (3.81, 80.0)
- moved XTAL1 1137.4 mm to (4.57, 85.6)
- moved R30 1125.8 mm to (52.8, 66.5), turned to 180 degrees
- moved R31 1125.6 mm to (52.8, 61.5)
- moved R29 1119.7 mm to (52.8, 65.0), turned to 180 degrees
- moved LED2 1114.1 mm to (59.9, 70.1)
- moved R28 1113.3 mm to (52.8, 63.2), turned to 180 degrees
- moved LED3 1110.4 mm to (45.5, 68.8), turned to 180 degrees
- moved LED5 1105.7 mm to (53.3, 59.2), turned to 180 degrees
- moved R24 1102.4 mm to (107.4, 86.1), turned to 90 degrees
- moved LED4 1099.8 mm to (52.8, 54.6), turned to 270 degrees
- moved R23 1098.6 mm to (110.2, 86.1), turned to 90 degrees
- moved TP3 1091.5 mm to (69.8, 57.9)
- moved TP6 1088.1 mm to (74.4, 43.2)
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Routing:
- net +12V: track 27.0 -> 33.2 mm
- net +5.000VREF: track 84.9 -> 83.7 mm
